Commit message: update existing urdfs to use meshes

File: src/kinematics/ur20.urdf (robot description, URDF)
Before this commit: robot ur20, 9 links, 7 joints
Links:
- added link ft_frame
- link base_link_inertia: mass None -> 4.0; geometry collision mesh filename=package://urdfs/ur20meshes/base.stl
- link forearm_link: mass None -> 7.879; geometry collision mesh filename=package://urdfs/ur20meshes/forearm.stl
- link shoulder_link: mass None -> 16.343; geometry collision mesh filename=package://urdfs/ur20meshes/shoulder.stl
- link upper_arm_link: mass None -> 29.632; geometry collision mesh filename=package://urdfs/ur20meshes/upperarm.stl
- link wrist_1_link: mass None -> 3.054; geometry collision mesh filename=package://urdfs/ur20meshes/wrist1.stl
- link wrist_2_link: mass None -> 3.126; geometry collision mesh filename=package://urdfs/ur20meshes/wrist2.stl
- link wrist_3_link: mass None -> 0.926; geometry collision mesh filename=package://urdfs/ur20meshes/wrist3.stl
Joints:
- added joint base_joint: type fixed, parent world, child base_link, origin xyz=0 0 0 rpy=0 0 3.141592653589793
- added joint wrist_3_link-ft_frame: type fixed, parent wrist_3_link, child ft_frame, origin xyz=0 0 0 rpy=0.0 0 0
- joint base_link-base_link_inertia: origin xyz=0 0 0 rpy=0 0 0 -> xyz=0 0 0 rpy=0 0 3.141592653589793

File: src/kinematics/ur5e.urdf (robot description, URDF)
Before this commit: robot ur5, 9 links, 8 joints
Links:
- removed link ee_link
- added link base_link_inertia, mass 4.0; collision mesh filename=package://urdfs/ur5emeshes/base.stl; visual mesh filename=package://ur_description/meshes/ur5e/visual/base.dae
- added link ft_frame
- link base_link: geometry 
- link forearm_link: mass None -> 2.846; geometry collision mesh filename=package://urdfs/ur5emeshes/forearm.stl; visual mesh filename=package://ur_description/meshes/ur5e/visual/forearm.dae
- link shoulder_link: mass None -> 3.761; geometry collision mesh filename=package://urdfs/ur5emeshes/shoulder.stl; visual mesh filename=package://ur_description/meshes/ur5e/visual/shoulder.dae
- link upper_arm_link: mass None -> 8.058; geometry collision mesh filename=package://urdfs/ur5emeshes/upperarm.stl; visual mesh filename=package://ur_description/meshes/ur5e/visual/upperarm.dae
- link wrist_1_link: mass None -> 1.37; geometry collision mesh filename=package://urdfs/ur5emeshes/wrist1.stl; visual mesh filename=package://ur_description/meshes/ur5e/visual/wrist1.dae
- link wrist_2_link: mass None -> 1.3; geometry collision mesh filename=package://urdfs/ur5emeshes/wrist2.stl; visual mesh filename=package://ur_description/meshes/ur5e/visual/wrist2.dae
- link wrist_3_link: mass None -> 0.365; geometry collision mesh filename=package://urdfs/ur5emeshes/wrist3.stl; visual mesh filename=package://ur_description/meshes/ur5e/visual/wrist3.dae
Joints:
- removed joint ee_joint
- added joint base_link-base_link_inertia: type fixed, parent base_link, child base_link_inertia, origin xyz=0 0 0 rpy=0 0 3.141592653589793
- added joint wrist_3_link-ft_frame: type fixed, parent wrist_3_link, child ft_frame, origin xyz=0 0 0 rpy=0.0 0 0
- joint base_joint: origin xyz=0.0 0.0 0.0 rpy=0.0 0.0 0.0 -> xyz=0 0 0 rpy=0 0 3.141592653589793
- joint elbow_joint: axis 0 -1 0 -> 0 0 1; limit lower=-3.141592 upper=3.141592 effort=150 velocity=3.141592 -> lower=-3.141592653589793 upper=3.141592653589793 effort=150.0 velocity=3.141592653589793; origin xyz=-0.425 0.0 0.0 rpy=0.0 0.0 0.0 -> xyz=-0.425 0 0 rpy=0 0 0
- joint shoulder_lift_joint: axis 0 -1 0 -> 0 0 1; limit lower=-6.283185 upper=6.283185 effort=150 velocity=3.141592 -> lower=-6.283185307179586 upper=6.283185307179586 effort=150.0 velocity=3.141592653589793; origin xyz=0.0 0.0 0.0 rpy=0.0 0.0 0.0 -> xyz=0 0 0 rpy=1.570796327 0 0
- joint shoulder_pan_joint: limit lower=-6.283185 upper=6.283185 effort=150 velocity=3.141592 -> lower=-6.283185307179586 upper=6.283185307179586 effort=150.0 velocity=3.141592653589793; origin xyz=0.0 0.0 0.1625 rpy=0.0 0.0 0.0 -> xyz=0 0 0.1625 rpy=0 0 0; parent base_link -> base_link_inertia
- joint wrist_1_joint: axis 0 -1 0 -> 0 0 1; limit lower=-6.283185 upper=6.283185 effort=28 velocity=3.141592 -> lower=-6.283185307179586 upper=6.283185307179586 effort=28.0 velocity=3.141592653589793; origin xyz=-.3922 -0.1333 0 rpy=0.0 0.0 0.0 -> xyz=-0.3922 0 0.1333 rpy=0 0 0
- joint wrist_2_joint: axis 0 0 -1 -> 0 0 1; limit lower=-6.283185 upper=6.283185 effort=28 velocity=3.141592 -> lower=-6.283185307179586 upper=6.283185307179586 effort=28.0 velocity=3.141592653589793; origin xyz=0.0 0.0 -0.0997 rpy=0.0 0.0 0.0 -> xyz=0 -0.0997 -2.044881182297852e-11 rpy=1.570796327 0 0
- joint wrist_3_joint: axis 0 -1 0 -> 0 0 1; limit lower=-6.283185 upper=6.283185 effort=28 velocity=3.141592 -> lower=-6.283185307179586 upper=6.283185307179586 effort=28.0 velocity=3.141592653589793; origin xyz=0.0 -0.0996 0.0 rpy=0.0 0.0 0.0 -> xyz=0 0.0996 -2.042830148012698e-11 rpy=1.570796326589793 3.141592653589793 3.141592653589793
